Commit message: lab 5

File: beginner_tutorials/urdf/robot.urdf (robot description, URDF)
Before this commit: robot fang, 5 links, 4 joints
Links:
- link link_0: geometry visual box size=0.9 0.5 0.5
- link link_1: geometry visual cylinder length=0.5 radius=0.4
- link link_2: geometry visual box size=2 0.4 0.4
- link link_3: geometry visual box size=0.2 0.7 0.6
Joints:
- joint base_joint: origin xyz=0.0 0.3 0.6 -> xyz=0.0 0 0
- joint joint_0: origin xyz=0 0 0 -> xyz=0 0 0.2
- joint joint_1: origin xyz=0.03 0.0 0.1 -> xyz=0 0.0 0.4
- joint joint_2: axis 0 0 1.1 -> 0 1 0; limit lower=-1 upper=1 effort=30 velocity=1.0 -> lower=-1 upper=1 effort=10 velocity=1.0; origin xyz=0.0 0 0 -> xyz= 0.5 0.5 1
